Commit message: feat: 完成 双臂URDF构建 moveit2双臂规划

File: ros2_rm_robot/rm_description/urdf/rm_75_macro.urdf.xacro (robot description, xacro)
@@ -1,10 +1,14 @@
 <?xml version="1.0" encoding="utf-8"?>
-<robot  name="rm_75_description" xmlns:xacro="http://www.ros.org/wiki/xacro">
+<robot xmlns:xacro="http://www.ros.org/wiki/xacro">
+  <xacro:macro name="rm_75_robot" params="prefix parent *origin">
+    <joint name="${prefix}base_joint" type="fixed">
+      <xacro:insert_block name="origin" />
+      <parent link="${parent}" />
+      <child link="${prefix}base_link" />
+    </joint>
 <!-- link6_type -->
-<xacro:arg name="link7_type" default="Link7" />
 <!-- arg->property -->
-<xacro:property name="link7_type" value="$(arg link7_type)" />
     <link
-    name="base_link">
+    name="${prefix}base_link">
     <inertial>
       <origin
@@ -46,5 +50,5 @@
   </link>
   <link
-    name="Link1">
+    name="${prefix}Link1">
     <inertial>
       <origin
@@ -86,5 +90,5 @@
   </link>
   <joint
-    name="joint1"
+    name="${prefix}joint1"
     type="revolute">
     <origin
@@ -92,7 +96,7 @@
       rpy="-1.5708 0 0" />
     <parent
-      link="base_link" />
-    <child
-      link="Link1" />
+      link="${prefix}base_link" />
+    <child
+      link="${prefix}Link1" />
     <axis
       xyz="0 -1 0" />
@@ -104,5 +108,5 @@
   </joint>
   <link
-    name="Link2">
+    name="${prefix}Link2">
     <inertial>
       <origin
@@ -144,5 +148,5 @@
   </link>
   <joint
-    name="joint2"
+    name="${prefix}joint2"
     type="revolute">
     <origin
@@ -150,7 +154,7 @@
       rpy="1.5708 0 0" />
     <parent
-      link="Link1" />
-    <child
-      link="Link2" />
+      link="${prefix}Link1" />
+    <child
+      link="${prefix}Link2" />
     <axis
       xyz="0 1 0" />
@@ -162,5 +166,5 @@
   </joint>
   <link
-    name="Link3">
+    name="${prefix}Link3">
     <inertial>
       <origin
@@ -202,5 +206,5 @@
   </link>
   <joint
-    name="joint3"
+    name="${prefix}joint3"
     type="revolute">
     <origin
@@ -208,7 +212,7 @@
       rpy="-1.5708 0 0" />
     <parent
-      link="Link2" />
-    <child
-      link="Link3" />
+      link="${prefix}Link2" />
+    <child
+      link="${prefix}Link3" />
     <axis
       xyz="0 -1 0" />
@@ -220,5 +224,5 @@
   </joint>
   <link
-    name="Link4">
+    name="${prefix}Link4">
     <inertial>
       <origin
@@ -260,5 +264,5 @@
   </link>
   <joint
-    name="joint4"
+    name="${prefix}joint4"
     type="revolute">
     <origin
@@ -266,7 +270,7 @@
       rpy="1.5708 0 0" />
     <parent
-      link="Link3" />
-    <child
-      link="Link4" />
+      link="${prefix}Link3" />
+    <child
+      link="${prefix}Link4" />
     <axis
       xyz="0 1 0" />
@@ -278,5 +282,5 @@
   </joint>
   <link
-    name="Link5">
+    name="${prefix}Link5">
     <inertial>
       <origin
@@ -318,5 +322,5 @@
   </link>
   <joint
-    name="joint5"
+    name="${prefix}joint5"
     type="revolute">
     <origin
@@ -324,7 +328,7 @@
       rpy="-1.5708 0 0" />
     <parent
-      link="Link4" />
-    <child
-      link="Link5" />
+      link="${prefix}Link4" />
+    <child
+      link="${prefix}Link5" />
     <axis
       xyz="0 -1 0" />
@@ -336,5 +340,5 @@
   </joint>
   <link
-    name="Link6">
+    name="${prefix}Link6">
     <inertial>
       <origin
@@ -376,5 +380,5 @@
   </link>
   <joint
-    name="joint6"
+    name="${prefix}joint6"
     type="revolute">
     <origin
@@ -382,7 +386,7 @@
       rpy="1.5708 0 0" />
     <parent
-      link="Link5" />
-    <child
-      link="Link6" />
+      link="${prefix}Link5" />
+    <child
+      link="${prefix}Link6" />
     <axis
       xyz="0 1 0" />
@@ -395,5 +399,5 @@
   <xacro:if value="${ link7_type =='Link7' }">
   <link
-    name="Link7">
+    name="${prefix}Link7">
     <inertial>
       <origin
@@ -435,5 +439,5 @@
   </link>
   <joint
-    name="joint7"
+    name="${prefix}joint7"
     type="revolute">
     <origin
@@ -441,7 +445,7 @@
       rpy="0 0 0" />
     <parent
-      link="Link6" />
-    <child
-      link="Link7" />
+      link="${prefix}Link6" />
+    <child
+      link="${prefix}Link7" />
     <axis
       xyz="0 0 1" />
@@ -455,5 +459,5 @@
   <xacro:if value="${ link7_type =='Link7_6f' }">
     <link
-    name="Link7">
+    name="${prefix}Link7">
     <inertial>
       <origin
@@ -495,5 +499,5 @@
   </link>
   <joint
-    name="joint7"
+    name="${prefix}joint7"
     type="revolute">
     <origin
@@ -501,7 +505,7 @@
       rpy="0 0 0" />
     <parent
-      link="Link6" />
-    <child
-      link="Link7" />
+      link="${prefix}Link6" />
+    <child
+      link="${prefix}Link7" />
     <axis
       xyz="0 0 1" />
@@ -515,5 +519,5 @@
     <xacro:if value="${ link7_type =='Link7_6fb' }">
     <link
-    name="Link7">
+    name="${prefix}Link7">
     <inertial>
       <origin
@@ -555,5 +559,5 @@
   </link>
   <joint
-    name="joint7"
+    name="${prefix}joint7"
     type="revolute">
     <origin
@@ -561,7 +565,7 @@
       rpy="0 0 0" />
     <parent
-      link="Link6" />
-    <child
-      link="Link7" />
+      link="${prefix}Link6" />
+    <child
+      link="${prefix}Link7" />
     <axis
       xyz="0 0 1" />
@@ -573,3 +577,4 @@
   </joint>
   </xacro:if>
+  </xacro:macro>
 </robot>
