Commit message: feat: 双臂 rviz+gazebo

File: ros2_rm_robot/rm_description/urdf/rm_75_dual.urdf.xacro (robot description, xacro)
@@ -31,3 +31,9 @@
     <origin xyz="0 -0.25 1.0" rpy="0 0 0"/>
   </xacro:rm_75_robot>
+  <gazebo>
+    <plugin filename="libgazebo_ros2_control.so" name="gazebo_ros2_control">
+      <parameters>$(find rm75_dual_config)/config/ros2_controllers.yaml</parameters>
+      <robot_param_node>robot_state_publisher</robot_param_node>
+    </plugin>
+  </gazebo>
 </robot>

File: ros2_rm_robot/rm_description/urdf/rm_75_macro.urdf.xacro (robot description, xacro)
@@ -31,19 +31,19 @@
       <geometry>
         <mesh
-          filename="package://rm_description/meshes/rm_75_arm/base_link.STL" />
-      </geometry>
-      <material
-        name="">
-        <color
-          rgba="1 1 1 1" />
-      </material>
-    </visual>
-    <collision>
-      <origin
-        xyz="0 0 0"
-        rpy="0 0 0" />
-      <geometry>
-        <mesh
-          filename="package://rm_description/meshes/rm_75_arm/base_link.STL" />
+          filename="file://$(find rm_description)/meshes/rm_75_arm/base_link.STL" />
+      </geometry>
+      <material
+        name="">
+        <color
+          rgba="1 1 1 1" />
+      </material>
+    </visual>
+    <collision>
+      <origin
+        xyz="0 0 0"
+        rpy="0 0 0" />
+      <geometry>
+        <mesh
+          filename="file://$(find rm_description)/meshes/rm_75_arm/base_link.STL" />
       </geometry>
     </collision>
@@ -71,19 +71,19 @@
       <geometry>
         <mesh
-          filename="package://rm_description/meshes/rm_75_arm/link1.STL" />
-      </geometry>
-      <material
-        name="">
-        <color
-          rgba="1 1 1 1" />
-      </material>
-    </visual>
-    <collision>
-      <origin
-        xyz="0 0 0"
-        rpy="0 0 0" />
-      <geometry>
-        <mesh
-          filename="package://rm_description/meshes/rm_75_arm/link1.STL" />
+          filename="file://$(find rm_description)/meshes/rm_75_arm/link1.STL" />
+      </geometry>
+      <material
+        name="">
+        <color
+          rgba="1 1 1 1" />
+      </material>
+    </visual>
+    <collision>
+      <origin
+        xyz="0 0 0"
+        rpy="0 0 0" />
+      <geometry>
+        <mesh
+          filename="file://$(find rm_description)/meshes/rm_75_arm/link1.STL" />
       </geometry>
     </collision>
@@ -129,19 +129,19 @@
       <geometry>
         <mesh
-          filename="package://rm_description/meshes/rm_75_arm/link2.STL" />
-      </geometry>
-      <material
-        name="">
-        <color
-          rgba="1 1 1 1" />
-      </material>
-    </visual>
-    <collision>
-      <origin
-        xyz="0 0 0"
-        rpy="0 0 0" />
-      <geometry>
-        <mesh
-          filename="package://rm_description/meshes/rm_75_arm/link2.STL" />
+          filename="file://$(find rm_description)/meshes/rm_75_arm/link2.STL" />
+      </geometry>
+      <material
+        name="">
+        <color
+          rgba="1 1 1 1" />
+      </material>
+    </visual>
+    <collision>
+      <origin
+        xyz="0 0 0"
+        rpy="0 0 0" />
+      <geometry>
+        <mesh
+          filename="file://$(find rm_description)/meshes/rm_75_arm/link2.STL" />
       </geometry>
     </collision>
@@ -187,19 +187,19 @@
       <geometry>
         <mesh
-          filename="package://rm_description/meshes/rm_75_arm/link3.STL" />
-      </geometry>
-      <material
-        name="">
-        <color
-          rgba="1 1 1 1" />
-      </material>
-    </visual>
-    <collision>
-      <origin
-        xyz="0 0 0"
-        rpy="0 0 0" />
-      <geometry>
-        <mesh
-          filename="package://rm_description/meshes/rm_75_arm/link3.STL" />
+          filename="file://$(find rm_description)/meshes/rm_75_arm/link3.STL" />
+      </geometry>
+      <material
+        name="">
+        <color
+          rgba="1 1 1 1" />
+      </material>
+    </visual>
+    <collision>
+      <origin
+        xyz="0 0 0"
+        rpy="0 0 0" />
+      <geometry>
+        <mesh
+          filename="file://$(find rm_description)/meshes/rm_75_arm/link3.STL" />
       </geometry>
     </collision>
@@ -245,19 +245,19 @@
       <geometry>
         <mesh
-          filename="package://rm_description/meshes/rm_75_arm/link4.STL" />
-      </geometry>
-      <material
-        name="">
-        <color
-          rgba="1 1 1 1" />
-      </material>
-    </visual>
-    <collision>
-      <origin
-        xyz="0 0 0"
-        rpy="0 0 0" />
-      <geometry>
-        <mesh
-          filename="package://rm_description/meshes/rm_75_arm/link4.STL" />
+          filename="file://$(find rm_description)/meshes/rm_75_arm/link4.STL" />
+      </geometry>
+      <material
+        name="">
+        <color
+          rgba="1 1 1 1" />
+      </material>
+    </visual>
+    <collision>
+      <origin
+        xyz="0 0 0"
+        rpy="0 0 0" />
+      <geometry>
+        <mesh
+          filename="file://$(find rm_description)/meshes/rm_75_arm/link4.STL" />
       </geometry>
     </collision>
@@ -303,19 +303,19 @@
       <geometry>
         <mesh
-          filename="package://rm_description/meshes/rm_75_arm/link5.STL" />
-      </geometry>
-      <material
-        name="">
-        <color
-          rgba="1 1 1 1" />
-      </material>
-    </visual>
-    <collision>
-      <origin
-        xyz="0 0 0"
-        rpy="0 0 0" />
-      <geometry>
-        <mesh
-          filename="package://rm_description/meshes/rm_75_arm/link5.STL" />
+          filename="file://$(find rm_description)/meshes/rm_75_arm/link5.STL" />
+      </geometry>
+      <material
+        name="">
+        <color
+          rgba="1 1 1 1" />
+      </material>
+    </visual>
+    <collision>
+      <origin
+        xyz="0 0 0"
+        rpy="0 0 0" />
+      <geometry>
+        <mesh
+          filename="file://$(find rm_description)/meshes/rm_75_arm/link5.STL" />
       </geometry>
     </collision>
@@ -361,19 +361,19 @@
       <geometry>
         <mesh
-          filename="package://rm_description/meshes/rm_75_arm/link6.STL" />
-      </geometry>
-      <material
-        name="">
-        <color
-          rgba="1 1 1 1" />
-      </material>
-    </visual>
-    <collision>
-      <origin
-        xyz="0 0 0"
-        rpy="0 0 0" />
-      <geometry>
-        <mesh
-          filename="package://rm_description/meshes/rm_75_arm/link6.STL" />
+          filename="file://$(find rm_description)/meshes/rm_75_arm/link6.STL" />
+      </geometry>
+      <material
+        name="">
+        <color
+          rgba="1 1 1 1" />
+      </material>
+    </visual>
+    <collision>
+      <origin
+        xyz="0 0 0"
+        rpy="0 0 0" />
+      <geometry>
+        <mesh
+          filename="file://$(find rm_description)/meshes/rm_75_arm/link6.STL" />
       </geometry>
     </collision>
@@ -420,19 +420,19 @@
       <geometry>
         <mesh
-          filename="package://rm_description/meshes/rm_75_arm/link7.STL" />
-      </geometry>
-      <material
-        name="">
-        <color
-          rgba="1 1 1 1" />
-      </material>
-    </visual>
-    <collision>
-      <origin
-        xyz="0 0 0"
-        rpy="0 0 0" />
-      <geometry>
-        <mesh
-          filename="package://rm_description/meshes/rm_75_arm/link7.STL" />
+          filename="file://$(find rm_description)/meshes/rm_75_arm/link7.STL" />
+      </geometry>
+      <material
+        name="">
+        <color
+          rgba="1 1 1 1" />
+      </material>
+    </visual>
+    <collision>
+      <origin
+        xyz="0 0 0"
+        rpy="0 0 0" />
+      <geometry>
+        <mesh
+          filename="file://$(find rm_description)/meshes/rm_75_arm/link7.STL" />
       </geometry>
     </collision>
@@ -480,19 +480,19 @@
       <geometry>
         <mesh
-          filename="package://rm_description/meshes/rm_75_arm/link7_6f.STL" />
-      </geometry>
-      <material
-        name="">
-        <color
-          rgba="1 1 1 1" />
-      </material>
-    </visual>
-    <collision>
-      <origin
-        xyz="0 0 0"
-        rpy="0 0 0" />
-      <geometry>
-        <mesh
-          filename="package://rm_description/meshes/rm_75_arm/link7_6f.STL" />
+          filename="file://$(find rm_description)/meshes/rm_75_arm/link7_6f.STL" />
+      </geometry>
+      <material
+        name="">
+        <color
+          rgba="1 1 1 1" />
+      </material>
+    </visual>
+    <collision>
+      <origin
+        xyz="0 0 0"
+        rpy="0 0 0" />
+      <geometry>
+        <mesh
+          filename="file://$(find rm_description)/meshes/rm_75_arm/link7_6f.STL" />
       </geometry>
     </collision>
@@ -540,5 +540,5 @@
       <geometry>
         <mesh
-          filename="package://rm_description/meshes/rm_75_arm/link7_6fb.STL" />
+          filename="file://$(find rm_description)/meshes/rm_75_arm/link7_6fb.STL" />
       </geometry>
       <material
@@ -554,5 +554,5 @@
       <geometry>
         <mesh
-          filename="package://rm_description/meshes/rm_75_arm/link7_6fb.STL" />
+          filename="file://$(find rm_description)/meshes/rm_75_arm/link7_6fb.STL" />
       </geometry>
     </collision>
@@ -577,4 +577,37 @@
   </joint>
   </xacro:if>
+  <ros2_control name="${prefix}GazeboSystem" type="system">
+      <hardware>
+        <plugin>gazebo_ros2_control/GazeboSystem</plugin>
+      </hardware>
+      <joint name="${prefix}joint1">
+        <command_interface name="position"><param name="min">-3.106</param><param name="max">3.106</param></command_interface>
+        <state_interface name="position"/><state_interface name="velocity"/>
+      </joint>
+      <joint name="${prefix}joint2">
+        <command_interface name="position"><param name="min">-2.268</param><param name="max">2.268</param></command_interface>
+        <state_interface name="position"/><state_interface name="velocity"/>
+      </joint>
+      <joint name="${prefix}joint3">
+        <command_interface name="position"><param name="min">-3.106</param><param name="max">3.106</param></command_interface>
+        <state_interface name="position"/><state_interface name="velocity"/>
+      </joint>
+      <joint name="${prefix}joint4">
+        <command_interface name="position"><param name="min">-2.356</param><param name="max">2.356</param></command_interface>
+        <state_interface name="position"/><state_interface name="velocity"/>
+      </joint>
+      <joint name="${prefix}joint5">
+        <command_interface name="position"><param name="min">-3.106</param><param name="max">3.106</param></command_interface>
+        <state_interface name="position"/><state_interface name="velocity"/>
+      </joint>
+      <joint name="${prefix}joint6">
+        <command_interface name="position"><param name="min">-2.233</param><param name="max">2.233</param></command_interface>
+        <state_interface name="position"/><state_interface name="velocity"/>
+      </joint>
+      <joint name="${prefix}joint7">
+        <command_interface name="position"><param name="min">-6.283</param><param name="max">6.283</param></command_interface>
+        <state_interface name="position"/><state_interface name="velocity"/>
+      </joint>
+  </ros2_control>
   </xacro:macro>
 </robot>
